Commit message: Robot with sensors in empty world

File: src/my_robot/urdf/my_robot.xacro (robot description, xacro)
@@ -1,4 +1,7 @@
 <?xml version='1.0'?>
 <robot name="my_robot" xmlns:xacro="http://www.ros.org/wiki/xacro">
+<!-- PLUGINS -->
+  <xacro:include filename="$(find my_robot)/urdf/my_robot.gazebo" />
+<!-- LINKS -->
   <link name="robot_footprint"></link>
   <link name='chassis'>
@@ -47,4 +50,86 @@
     </visual>
   </link>
+  <link name='right_wheel'>
+    <pose>0 0 0 0 0 0 0</pose>
+    <inertial>
+      <mass value="5" />
+      <origin xyz="0 0 0" rpy="0 1.5707 1.5707" />
+      <inertia ixx="0.1" ixy="0" ixz="0" iyy="0.1" iyz="0" izz="0.1" />
+    </inertial>
+    <collision name='right_wheel_collision'>
+      <origin xyz="0 0 0" rpy="0 1.5707 1.5707" />
+      <geometry>
+        <cylinder radius="0.1" length="0.05" />
+      </geometry>
+    </collision>
+    <visual name='right_wheel_visual'>
+      <origin xyz="0 0 0" rpy="0 1.5707 1.5707" />
+      <geometry>
+        <cylinder radius="0.1" length="0.05" />
+      </geometry>
+    </visual>
+  </link>
+  <link name='left_wheel'>
+    <pose>0 0 0 0 0 0 0</pose>
+    <inertial>
+      <mass value="5" />
+      <origin xyz="0 0 0" rpy="0 1.5707 1.5707" />
+      <inertia ixx="0.1" ixy="0" ixz="0" iyy="0.1" iyz="0" izz="0.1" />
+    </inertial>
+    <collision name='left_wheel_collision'>
+      <origin xyz="0 0 0" rpy="0 1.5707 1.5707" />
+      <geometry>
+        <cylinder radius="0.1" length="0.05" />
+      </geometry>
+    </collision>
+    <visual name='left_wheel_visual'>
+      <origin xyz="0 0 0" rpy="0 1.5707 1.5707" />
+      <geometry>
+        <cylinder radius="0.1" length="0.05" />
+      </geometry>
+    </visual>
+  </link>
+<!-- SENSORS -->
+  <link name="camera">
+    <pose>0 0 0 0 0 0</pose>
+    <inertial>
+      <mass value="0.1" />
+      <origin xyz="0 0 0" rpy="0 0 0" />
+      <inertia ixx="1e-6" ixy="0" ixz="0" iyy="1e-6" iyz="0" izz="1e-6" />
+    </inertial>
+    <collision name="camera_collision">
+      <origin xyz="0 0 0" rpy="0 0 0" />
+      <geometry>
+        <box size="0.05 0.05 0.05" />
+      </geometry>
+    </collision>
+    <visual name="camera_visual">
+      <origin xyz="0 0 0" rpy="0 0 0" />
+      <geometry>
+        <box size="0.05 0.05 0.05" />
+      </geometry>
+    </visual>
+  </link>
+  <link name="hokuyo">
+    <pose>0 0 0 0 0 0</pose>
+    <inertial>
+      <mass value="1e-5" />
+      <origin xyz="0 0 0" rpy="0 0 0" />
+      <inertia ixx="1e-6" ixy="0" ixz="0" iyy="1e-6" iyz="0" izz="1e-6" />
+    </inertial>
+    <collision name="camera_collision">
+      <origin xyz="0 0 0" rpy="0 0 0" />
+      <geometry>
+        <box size="0.1 0.1 0.1" />
+      </geometry>
+    </collision>
+    <visual name="camera_visual">
+      <origin xyz="0 0 0" rpy="0 0 0" />
+      <geometry>
+        <mesh filename="package://my_robot/meshes/hokuyo.dae" />
+      </geometry>
+    </visual>
+  </link>
+<!-- JOINTS -->
   <joint name="robot_footprint_joint" type="fixed">
     <origin xyz="0 0 0" rpy="0 0 0" />
@@ -52,3 +137,44 @@
     <child link="chassis" />
   </joint>
+  <joint name="right_wheel_hinge" type="continuous">
+    <origin xyz="0 0.15 0" rpy="0 0 0" />
+    <parent link="chassis" />
+    <child link="right_wheel" />
+    <axis xyz="0 1 0" rpy="0 0 0" />
+    <limit effort="10000" velocity="1000" />
+    <dynamics damping="1.0" friction="1.0" />
+  </joint>
+  <joint name="left_wheel_hinge" type="continuous">
+    <origin xyz="0 -0.15 0" rpy="0 0 0" />
+    <parent link="chassis" />
+    <child link="left_wheel" />
+    <axis xyz="0 1 0" rpy="0 0 0" />
+    <limit effort="10000" velocity="1000" />
+    <dynamics damping="1.0" friction="1.0" />
+  </joint>
+  <joint name="camera_joint" type="fixed">
+    <origin xyz="0.2 0 0" rpy="0 0 0" />
+    <parent link="chassis" />
+    <child link="camera" />
+    <axis xyz="0 1 0" rpy="0 0 0" />
+  </joint>
+  <joint name="hokuyo_joint" type="fixed">
+    <origin xyz="0.15 0 0.1" rpy="0 0 0" />
+    <parent link="chassis" />
+    <child link="hokuyo" />
+    <axis xyz="0 1 0" rpy="0 0 0" />
+  </joint>
+<!-- GAZEBO ELEMENTS -->
+  <gazebo reference="left_wheel">
+    <material>Gazebo/Black</material>
+  </gazebo>
+  <gazebo reference="right_wheel">
+    <material>Gazebo/Black</material>
+  </gazebo>
+  <gazebo reference="chassis">
+    <material>Gazebo/DarkYellow</material>
+  </gazebo>
+  <gazebo reference="camera">
+    <material>Gazebo/DarkGrey</material>
+  </gazebo>
 </robot>
